Commit message: speed and torque command interfaces, standard controllers, jtc test

File: realhand_l6_description/urdf/realhand_l6.ros2_control.xacro (robot description, xacro)
@@ -13,8 +13,10 @@
     enable_tactile request taxel matrices from the hand
     taxel_topic    when set, the driver publishes raw taxel grids there
+    setpoints      add speed and torque command interfaces (raw 0 to 255)
+                   to every actuated joint, default true
 -->
 <robot xmlns:xacro="http://www.ros.org/wiki/xacro">
   <xacro:macro name="realhand_l6_ros2_control"
-    params="name prefix:='' side:=right hardware:=mock can_interface:=can0 can_id:='' enable_tactile:=true taxel_topic:=''">
+    params="name prefix:='' side:=right hardware:=mock can_interface:=can0 can_id:='' enable_tactile:=true taxel_topic:='' setpoints:=true">
     <xacro:macro name="actuated" params="joint upper">
       <joint name="${prefix}${joint}">
@@ -23,4 +25,14 @@
           <param name="max">${upper}</param>
         </command_interface>
+        <xacro:if value="${setpoints}">
+          <command_interface name="speed">
+            <param name="min">0</param>
+            <param name="max">255</param>
+          </command_interface>
+          <command_interface name="torque">
+            <param name="min">0</param>
+            <param name="max">255</param>
+          </command_interface>
+        </xacro:if>
         <state_interface name="position">
           <param name="initial_value">0.0</param>

File: realhand_l6_description/urdf/realhand_l6.urdf.xacro (robot description, xacro)
@@ -10,4 +10,5 @@
     enable_tactile request taxel matrices from the hand
     taxel_topic    optional raw taxel JSON topic
+    setpoints      speed and torque command interfaces on actuated joints
 -->
 <robot xmlns:xacro="http://www.ros.org/wiki/xacro" name="realhand_l6">
@@ -19,4 +20,5 @@
   <xacro:arg name="enable_tactile" default="true"/>
   <xacro:arg name="taxel_topic" default=""/>
+  <xacro:arg name="setpoints" default="true"/>
   <xacro:include filename="realhand_l6_macro.xacro"/>
   <xacro:include filename="realhand_l6.ros2_control.xacro"/>
@@ -34,5 +36,6 @@
       can_id="$(arg can_id)"
       enable_tactile="$(arg enable_tactile)"
-      taxel_topic="$(arg taxel_topic)"/>
+      taxel_topic="$(arg taxel_topic)"
+      setpoints="$(arg setpoints)"/>
   </xacro:unless>
 </robot>

File: realhand_l6_description/urdf/realhand_l6_macro.xacro (robot description, xacro)
@@ -221,5 +221,5 @@
       <child link="${prefix}thumb_metacarpals_base2"/>
       <axis xyz="0 0 ${-reflect}"/>
-      <limit lower="-0.01" upper="1.54" effort="100" velocity="1"/>
+      <limit lower="0" upper="1.54" effort="100" velocity="1"/>
       <dynamics damping="0.1"/>
     </joint>
@@ -229,5 +229,5 @@
       <child link="${prefix}thumb_metacarpals"/>
       <axis xyz="0 1 0"/>
-      <limit lower="-0.01" upper="0.52" effort="100" velocity="1"/>
+      <limit lower="0" upper="0.52" effort="100" velocity="1"/>
       <dynamics damping="0.1"/>
     </joint>
@@ -246,5 +246,5 @@
       <child link="${prefix}index_proximal"/>
       <axis xyz="0 1 0"/>
-      <limit lower="-0.01" upper="1.57" effort="100" velocity="1"/>
+      <limit lower="0" upper="1.57" effort="100" velocity="1"/>
       <dynamics damping="0.1"/>
     </joint>
@@ -254,5 +254,5 @@
       <child link="${prefix}index_distal"/>
       <axis xyz="0 1 0"/>
-      <limit lower="-0.01" upper="1.4" effort="100" velocity="1"/>
+      <limit lower="0" upper="1.4" effort="100" velocity="1"/>
       <dynamics damping="0.1"/>
       <mimic joint="${prefix}index_mcp_pitch" multiplier="0.89" offset="0"/>
@@ -263,5 +263,5 @@
       <child link="${prefix}middle_proximal"/>
       <axis xyz="0 1 0"/>
-      <limit lower="-0.01" upper="1.57" effort="100" velocity="1"/>
+      <limit lower="0" upper="1.57" effort="100" velocity="1"/>
       <dynamics damping="0.1"/>
     </joint>
@@ -271,5 +271,5 @@
       <child link="${prefix}middle_distal"/>
       <axis xyz="0 1 0"/>
-      <limit lower="-0.01" upper="1.4" effort="100" velocity="1"/>
+      <limit lower="0" upper="1.4" effort="100" velocity="1"/>
       <dynamics damping="0.1"/>
       <mimic joint="${prefix}middle_mcp_pitch" multiplier="0.89" offset="0"/>
@@ -280,5 +280,5 @@
       <child link="${prefix}ring_proximal"/>
       <axis xyz="0 1 0"/>
-      <limit lower="-0.01" upper="1.57" effort="100" velocity="1"/>
+      <limit lower="0" upper="1.57" effort="100" velocity="1"/>
       <dynamics damping="0.1"/>
     </joint>
@@ -288,5 +288,5 @@
       <child link="${prefix}ring_distal"/>
       <axis xyz="0 1 0"/>
-      <limit lower="-0.01" upper="1.4" effort="100" velocity="1"/>
+      <limit lower="0" upper="1.4" effort="100" velocity="1"/>
       <dynamics damping="0.1"/>
       <mimic joint="${prefix}ring_mcp_pitch" multiplier="0.89" offset="0"/>
@@ -297,5 +297,5 @@
       <child link="${prefix}pinky_proximal"/>
       <axis xyz="0 1 0"/>
-      <limit lower="-0.01" upper="1.57" effort="100" velocity="1"/>
+      <limit lower="0" upper="1.57" effort="100" velocity="1"/>
       <dynamics damping="0.1"/>
     </joint>
@@ -305,5 +305,5 @@
       <child link="${prefix}pinky_distal"/>
       <axis xyz="0 1 0"/>
-      <limit lower="-0.01" upper="1.4" effort="100" velocity="1"/>
+      <limit lower="0" upper="1.4" effort="100" velocity="1"/>
       <dynamics damping="0.1"/>
       <mimic joint="${prefix}pinky_mcp_pitch" multiplier="0.89" offset="0"/>
